File: ETAG.brd (EAGLE design)
At the start: 68.6 x 53.3 mm, 98 parts, among them CN2 PINHEAD-2x5-P1.27, IC2 SAMD21G18A-AUT, IC5 RTC_PCF8523T, IC6 EM4095, K1 G3VM-202J1, K2 G3VM-202J1, U2 TC7SU04F, Y1 32.768kHz, Y4 32,768Khz

Commit message: Added 3.3V LDO regulator for USB power
Parts:
- removed D3, D4: (no value), diode:LL-34
- removed D5: M7, Diodi:SMB
- removed TP_0, TP_1, TP_2, TP_3, TP_4, TP_5, TP_6, TP_7, TP_8, TP_9: TP_SP, SmartPrj:TP-SP
- added C2: 1u, Condensatori:C0603-ROUND
- added C6: 4.7u, Condensatori:C0603-ROUND
- added J1: 22-27-2021-02, con-molex:6410-02
- added T1_VDIV, T_SD: P_CHANNEL_MOSFET_, transistor-fet:SOT23
- added U$1: MCP1824T-3302E/OT, Microchip_By_element14_Batch_1:SOT95P270X145-5N
- added VDIV1, VDIV2, VDIV_USB: ?, Resistenze:R0603-ROUND
- moved LED1 33.2 mm to (7.62, 1.65), turned to 90 degrees
- moved R6 28.7 mm to (7.75, 3.43)
- moved R5 3.47 mm to (23.9, 18.8), turned to 90 degrees
- moved C_CO1 3.14 mm to (41.0, 8.38)
- moved L1 3.10 mm to (44.6, 15.0)
- moved FD2 2.67 mm to (2.31, 2.13)
- moved IC6 2.29 mm to (29.3, 34.4)
- moved CRES 2.25 mm to (22.9, 31.9)
- moved CDIV1 2.22 mm to (22.9, 29.5)
- moved CDIV2 2.19 mm to (22.9, 27.1)
- moved CAGND 2.04 mm to (34.4, 33.3)
- moved R7 1.91 mm to (23.0, 36.8)
- moved CFCAP 1.61 mm to (35.2, 37.5), turned to 0 degrees
- moved C_BST 1.57 mm to (34.7, 22.1)
- moved C_VC1 1.40 mm to (27.9, 19.1)
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Connections:
- removed net DGI_GPIO1: TP_7.X
- removed net DGI_GPIO2_PA6: IC2.11, IOH.1, TP_8.X
- removed net DGI_GPIO3_PA7: IC2.12, IOH.2, K2.1, K2.3, TP_9.X, U2.2
- removed net N$21: D5.A, U$9.P$1
- removed net N$24: D3.P$2, D4.P$2, R5.1
- removed net PA21_RTC_INT: IC2.30, IC5.7, R9.1
- removed net PA28_SD_CS: IC2.41, U$4.1
- removed net PB22_RFID_RDY: IC2.37, IC6.2
- removed net PB23_RFID_SHD: IC2.38, IC6.14
- removed net PWRIN_1: U$6.P$1, U$6.P$2, U$9.P$3
- removed net VIN: C_VC1.2, D4.P$1, D5.C, POWER.8, U$3.4
- new net +12V: C_VC1.2, POWER.8, R5.1, T1_VDIV.2, U$3.4, U$6.P$3, U$6.P$4
- new net +3.3_PSU: C_CO2.2, C_UP.1, L2.2, R-UP.2, U$9.P$5
- new net +5_PSU: C_CO1.1, C_CO3.1, L1.P$1, U$3.8, U$9.P$6
- new net N$23: T1_VDIV.3, VDIV2.2
- new net PA06_AIN6: IC2.11, IOH.1
- new net PA19_MISO: IC2.28, IOH.5
- new net PA21_INT&SDCS: IC2.30, IC5.7, R9.1, U$4.1
- new net PA28_2FETS: IC2.41, T1_VDIV.1, T_SD.1
- new net PA6_RFID_SHD: IC6.14
- new net PA7_RF_SWTICH: IC2.12, IOH.2, K2.1, K2.3, U2.2
- new net PB22_DEBUG_TX: IC2.37, J1.2
- new net PB23_DEBUG_RX: IC2.38, J1.1
- new net VDD: T_SD.3, U$4.4
- new net X3.3V: C2.2, U$1.5, U$9.P$1, VDIV_USB.2
- net +3V3: now also T_SD.2, U$9.P$3; no longer C_CO2.2, C_UP.1, L2.2, R-UP.2, U$4.4
- net +5V: now also U$9.P$4; no longer C_CO1.1, C_CO3.1, D3.P$1, L1.P$1, U$3.8, U$9.P$6
- net GND: now also C2.1, C6.1, U$1.2, U$6.P$1, U$6.P$2, VDIV1.1; no longer U$6.P$3, U$6.P$4
- net PA02_AIN0: now also VDIV1.2, VDIV2.1, VDIV_USB.1
- net PA08_TCC0-W0_PA8: no longer TP_2.X
- net PA09_TCC0-W1_PA9: no longer TP_3.X
- net PA10_MISO: no longer IC2.28, IOH.5
- net PA10_TCC0-W2_PA10: no longer TP_1.X
- net PA11_TCC0-W3_PA11: no longer TP_0.X
- net PA14_TCC0-W4: no longer TP_4.X
- net PA15_TCC0-W5: no longer TP_5.X
- net PA20_TCC0-W6: no longer TP_6.X
- net XUSB: now also C6.2, U$1.1, U$1.3, U$9.P$2; no longer U$9.P$4
Routing:
- net DGI_GPIO3_PA7: track 68.2 -> 0.00 mm, vias 3 -> 0
- net PA7_RF_SWTICH: track 0.00 -> 67.7 mm, vias 0 -> 3
- net +5V: track 179.4 -> 121.3 mm, vias 1 -> 4
- net PA28_2FETS: track 0.00 -> 54.4 mm, vias 0 -> 3
- net VIN: track 53.4 -> 0.00 mm, vias 1 -> 0
- net +12V: track 0.00 -> 52.1 mm, vias 0 -> 1
- net PA02_AIN0: track 40.9 -> 89.9 mm, vias 0 -> 1
- net PA21_INT&SDCS: track 0.00 -> 39.6 mm, vias 0 -> 1
- net PA28_SD_CS: track 28.7 -> 0.00 mm, vias 1 -> 0
- net PA19_MISO: track 0.00 -> 24.9 mm
- net PA10_MISO: track 25.0 -> 0.05 mm
- net PB23_RFID_SHD: track 23.7 -> 0.00 mm, vias 2 -> 0
- net PB22_RFID_RDY: track 22.9 -> 0.00 mm, vias 2 -> 0
- net PA06_AIN6: track 0.00 -> 22.3 mm, vias 0 -> 1
- net DGI_GPIO2_PA6: track 22.2 -> 0.00 mm, vias 1 -> 0
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