File: ETAG.sch (EAGLE design)
At the start: 98 parts, among them CN2 PINHEAD-2x5-P1.27, IC2 SAMD21G18A-AUT, IC5 RTC_PCF8523T, IC6 EM4095, K1 G3VM-202J1, K2 G3VM-202J1, U2 TC7SU04F, Y1 32.768kHz, Y4 32,768Khz

Commit message: Added 3.3V LDO regulator for USB power
Parts:
- removed D3, D4: (no value), diode:DIODE-LL-34
- removed D5: M7, Diodi:0020_M7
- removed TP_0, TP_1, TP_2, TP_3, TP_4, TP_5, TP_6, TP_7, TP_8, TP_9: TP_SP, SmartPrj:TP_SP
- added C2: 1u, Condensatori:0142_10NF_0603
- added C6: 4.7u, Condensatori:0142_10NF_0603
- added J1: 22-27-2021-02, con-molex:22-27-2021-02
- added T1_VDIV, T_SD: P_CHANNEL_MOSFET_, transistor-fet:P_CHANNEL_MOSFET_
- added U$1: MCP1824T-3302E/OT, Microchip_By_element14_Batch_1:MCP1824T-3302E/OT
- added VDIV1, VDIV_USB: ?, Resistenze:2339_
- added VDIV2: ?, Resistenze:2022_CR0603FW104L
Connections:
- removed net DGI_GPIO1: TP_7.TESTP
- removed net DGI_GPIO2_PA6: IC2.PA6/EIC/AIN6/SCOM0PAD2/TC1, IOH.1, TP_8.TESTP
- removed net DGI_GPIO3_PA7: IC2.PA7/EIC/AIN7/SCOM0PAD3/TC1, IOH.2, K2-1.A, K2-2.A, TP_9.TESTP, U2.A
- removed net N$21: D5.A, U$9.O
- removed net N$24: D3.C, D4.C, R5.1
- removed net PA21_RTC_INT: IC2.PA21/EIC/SCOM5PAD3+, IC5.!INT1/CLK, R9.1
- removed net PA28_SD_CS: IC2.PA28/EIC, U$4.CS
- removed net PB22_RFID_RDY: IC2.PB22/EIC/SCOM5PAD2, IC6.RDY/CLK
- removed net PB23_RFID_SHD: IC2.PB23/EIC/SCOM5PAD3, IC6.SHD
- removed net PWRIN_1: U$6G$1.S, U$9.P
- removed net VIN: C_VC1.2, D4.A, D5.C, POWER.8, U$3.P4_VIN
- new net +12V: C_VC1.2, POWER.8, R5.1, T1_VDIV.S, U$3.P4_VIN, U$6G$2.S
- new net +3.3_PSU: C_CO2.2, C_UP.1, L2.2, R-UP.2, U$9.S
- new net +5_PSU: C_CO1.1, C_CO3.1, L1.1, U$3.P8_VO, U$9.S1
- new net N$23: T1_VDIV.D, VDIV2.2
- new net PA06_AIN6: IC2.PA6/EIC/AIN6/SCOM0PAD2/TC1, IOH.1
- new net PA19_MISO: IC2.PA19/EIC/SCOM1PAD3+/TC3, IOH.5
- new net PA21_INT&SDCS: IC2.PA21/EIC/SCOM5PAD3+, IC5.!INT1/CLK, R9.1, U$4.CS
- new net PA28_2FETS: IC2.PA28/EIC, T1_VDIV.G, T_SD.G
- new net PA6_RFID_SHD: IC6.SHD
- new net PA7_RF_SWTICH: IC2.PA7/EIC/AIN7/SCOM0PAD3/TC1, IOH.2, K2-1.A, K2-2.A, U2.A
- new net PB22_DEBUG_TX: IC2.PB22/EIC/SCOM5PAD2, J1-2.S
- new net PB23_DEBUG_RX: IC2.PB23/EIC/SCOM5PAD3, J1-1.S
- new net VDD: T_SD.D, U$4.VDD
- new net X3.3V: C2.2, U$1.VOUT, U$9.O, VDIV_USB.2
- net +3V3: now also T_SD.S, U$9.P; no longer C_CO2.2, C_UP.1, L2.2, R-UP.2, U$4.VDD
- net +5V: now also U$9.P1; no longer C_CO1.1, C_CO3.1, D3.A, L1.1, U$3.P8_VO, U$9.S1
- net GND: now also C2.1, C6.1, U$1.GND, U$6G$1.S, VDIV1.1; no longer U$6G$2.S
- net PA02_AIN0: now also VDIV1.2, VDIV2.1, VDIV_USB.1
- net PA08_TCC0-W0_PA8: no longer TP_2.TESTP
- net PA09_TCC0-W1_PA9: no longer TP_3.TESTP
- net PA10_MISO: no longer IC2.PA19/EIC/SCOM1PAD3+/TC3, IOH.5
- net PA10_TCC0-W2_PA10: no longer TP_1.TESTP
- net PA11_TCC0-W3_PA11: no longer TP_0.TESTP
- net PA14_TCC0-W4: no longer TP_4.TESTP
- net PA15_TCC0-W5: no longer TP_5.TESTP
- net PA20_TCC0-W6: no longer TP_6.TESTP
- net XUSB: now also C6.2, U$1.VIN, U$1.~SHDN, U$9.O1; no longer U$9.P1
Other:
- moved on the sheet: C19, C20, CAGND, CDC2, CDEC, CRES, R7, U$6G$1, U$6G$2, U$9
